File: circuit schematics/PKM_MAN_IC_AC.kicad_sch (KiCad schematic)
At the start: 10 parts

Commit message: multimeter
Parts:
- removed HOLD: Hold_Button, symbol Connector:Conn_01x02_Pin
- removed INPUT (x2): Input_Vol, symbol Connector:Screw_Terminal_01x02
- removed OUTPUT (x2): DC_Vol, symbol Connector:Conn_01x03_Socket
- removed RST: Reset_Button, symbol Connector:Conn_01x02_Pin
- added HOLD_BUTTON, RESET_BUTTON: SW_Push, symbol Switch:SW_Push
- added INPUT (x2): Input_Vol, symbol Connector:Screw_Terminal_01x02
- added OUTPUT: DC_Vol, symbol Connector:Conn_01x03_Socket
- added OUTPUT: Conn_01x04_Socket, symbol Connector:Conn_01x04_Socket
Connections:
- net GND: now also HOLD_BUTTON.2, OUTPUT.3 (Pin_3), OUTPUT.3 (Pin_3), OUTPUT.4 (Pin_4), RESET_BUTTON.2
- net HOLD: now also HOLD_BUTTON.1
- net Input_GND: now also INPUT.1 (Pin_1), INPUT.1 (Pin_1)
- net Input_VCC: now also INPUT.2 (Pin_2), INPUT.2 (Pin_2)
- net RESET: now also RESET_BUTTON.1
- net SIG_A: now also OUTPUT.2 (Pin_2)
- net SIG_V: now also OUTPUT.2 (Pin_2)
- net VCC_5V: now also OUTPUT.1 (Pin_1), OUTPUT.1 (Pin_1)
Other:
- note added: "AC CURRENT SENSOR"
- note added: "AC VOLTAGE SENSOR"
- note added: "PKM MAN IC AC CIRCUIT SCHEMATIC"
- note removed: "DC CURRENT SENSOR"
- note removed: "DC VOLTAGE SENSOR"
- note removed: "PKM MAN IC DC CIRCUIT SCHEMATIC"
